Commit message: removed dependencies

File: urdf/arm.xacro (robot description, xacro)
@@ -1,7 +1,7 @@
 <?xml version="1.0"?>
 <robot name="arm" xmlns:xacro="http://www.ros.org/wiki/xacro">
-  <xacro:include filename="$(find arm_description)/urdf/materials.xacro" />
-  <xacro:include filename="$(find arm_description)/urdf/arm.trans" />
-  <xacro:include filename="$(find arm_description)/urdf/arm.gazebo" />
+  <xacro:include filename="$(find SPARK-A-4DOF-ROS-ROBOTIC-ARM)/urdf/materials.xacro" />
+  <xacro:include filename="$(find SPARK-A-4DOF-ROS-ROBOTIC-ARM)/urdf/arm.trans" />
+  <xacro:include filename="$(find SPARK-A-4DOF-ROS-ROBOTIC-ARM)/urdf/arm.gazebo" />
   <!-- World link -->
   <link name="world"></link>
@@ -37,5 +37,5 @@
       <origin xyz="0 0 0" rpy="0 0 0" />
       <geometry>
-        <mesh filename="package://arm_description/meshes/base_link.stl" scale="0.01 0.01 0.01" />
+        <mesh filename="package://SPARK-A-4DOF-ROS-ROBOTIC-ARM/meshes/base_link.stl" scale="0.01 0.01 0.01" />
       </geometry>
       <material name="silver" />
@@ -44,5 +44,5 @@
       <origin xyz="0 0 0" rpy="0 0 0" />
       <geometry>
-        <mesh filename="package://arm_description/meshes/base_link.stl" scale="0.01 0.01 0.01" />
+        <mesh filename="package://SPARK-A-4DOF-ROS-ROBOTIC-ARM/meshes/base_link.stl" scale="0.01 0.01 0.01" />
       </geometry>
     </collision>
@@ -58,5 +58,5 @@
       <origin xyz="0.05 0 -0.3" rpy="0 0 0" />
       <geometry>
-        <mesh filename="package://arm_description/meshes/Link_A_1.stl" scale="0.01 0.01 0.01" />
+        <mesh filename="package://SPARK-A-4DOF-ROS-ROBOTIC-ARM/meshes/Link_A_1.stl" scale="0.01 0.01 0.01" />
       </geometry>
       <material name="silver" />
@@ -65,5 +65,5 @@
       <origin xyz="0.05 -0.0 -0.3" rpy="0 0 0" />
       <geometry>
-        <mesh filename="package://arm_description/meshes/Link_A_1.stl" scale="0.01 0.01 0.01" />
+        <mesh filename="package://SPARK-A-4DOF-ROS-ROBOTIC-ARM/meshes/Link_A_1.stl" scale="0.01 0.01 0.01" />
       </geometry>
     </collision>
@@ -79,5 +79,5 @@
       <origin xyz="0.05 -0.0 -1.05" rpy="0 0 0" />
       <geometry>
-        <mesh filename="package://arm_description/meshes/Link_B_1.stl" scale="0.01 0.01 0.01" />
+        <mesh filename="package://SPARK-A-4DOF-ROS-ROBOTIC-ARM/meshes/Link_B_1.stl" scale="0.01 0.01 0.01" />
       </geometry>
       <material name="silver" />
@@ -86,5 +86,5 @@
       <origin xyz="0.05 0.0 -1.05" rpy="0 0 0" />
       <geometry>
-        <mesh filename="package://arm_description/meshes/Link_B_1.stl" scale="0.01 0.01 0.01" />
+        <mesh filename="package://SPARK-A-4DOF-ROS-ROBOTIC-ARM/meshes/Link_B_1.stl" scale="0.01 0.01 0.01" />
       </geometry>
     </collision>
@@ -100,5 +100,5 @@
       <origin xyz="-0.1 0.0 0.25" rpy="0 0 0" />
       <geometry>
-        <mesh filename="package://arm_description/meshes/end_effector.stl" scale="0.01 0.01 0.01" />
+        <mesh filename="package://SPARK-A-4DOF-ROS-ROBOTIC-ARM/meshes/end_effector.stl" scale="0.01 0.01 0.01" />
       </geometry>
       <material name="silver" />
@@ -107,5 +107,5 @@
       <origin xyz="-0.1 0.0 0.25" rpy="0 0 0" />
       <geometry>
-        <mesh filename="package://arm_description/meshes/end_effector.stl" scale="0.01 0.01 0.01" />
+        <mesh filename="package://SPARK-A-4DOF-ROS-ROBOTIC-ARM/meshes/end_effector.stl" scale="0.01 0.01 0.01" />
       </geometry>
     </collision>
